Commit message: first update

File: src/robot_drive/description/robot.urdf.xacro (robot description, xacro)
@@ -10,3 +10,4 @@
         <xacro:include filename="gazebo_control.xacro" />
     </xacro:unless>
+    <xacro:include filename="lidar.xacro" />
 </robot>

File: src/robot_drive/description/ros2_control.xacro (robot description, xacro)
@@ -52,8 +52,8 @@
                 <state_interface name="position"/>
             </joint>
-            <joint name="chassis">
+            <!-- <joint name="chassis_joint">
                 <state_interface name="velocity"/>
                 <state_interface name="position"/>
-            </joint>
+            </joint> -->
         </ros2_control>
     </xacro:if>
